Commit message: feat: replace the TG-9801 gripper with a LinkerHand O6
Change the deployment's body from the TG-9801 adaptive gripper to a
LinkerHand O6 six-axis dexterous hand on the JAKA controller's end RS485L
channel. The controller allows only one active jkrc session and its RS485
signal table is global, so the arm and the hand cannot be two processes:
the deployment now uses one combined primitive
(primitive-jaka-mini_with_linker_hand_o6-arm_hand-rbnx) that serves both
contract families.

- soma.yaml: the gripper component becomes an `end_effector` hand served
  by jaka_arm through robonix/primitive/hand/{info,move_joint,state_joint,
  set_joint_*_limits}; no gripper state aggregation (a six-actuator hand is
  not a single open/close joint).
- urdf/robot.urdf: the TG-9801 finger chain (link_008/link_009 + prismatic
  joints) is replaced by the O6 chain (17 links, 6 actuated joints, 5 mimic
  distal joints, meshes/right_hand/). link_007_to_hand is a PLACEHOLDER
  pose pending on-site measurement.
- robonix_manifest.yaml: jaka_arm points at the combined arm+hand package
  with end_effector: hand / hand_type: right; the separate hand primitive
  is dropped. The skill keeps its original six capabilities; its heights
  move to the O6 palm (desktop 0.14, hover 0.29, pick travel 0.08) and
  gripper_settle_s is raised to 3 s.
- tools/calibration: drives the O6 open/grip through the combined driver,
  probes the new package and uses the 0.14 m desktop height.
- README: single-jkrc-session architecture, hand contracts, the unchanged
  skill's gripper_joint mapping and the updated acceptance flow.

Bench-verified 2026-10-22: one jkrc session for both families, 12-joint
joint_states, hand/info + move_joint + the unknown-pose guard, the skill's
gripper_joint open/grip path, and healthy arm feedback while the hand moved.

Assisted-by: DeepSeek-Harness:deepseek-flash

File: urdf/robot.urdf (robot description, URDF)
Before this commit: robot generated_robot, 9 links, 8 joints
Links:
- removed link link_008
- removed link link_009
- added link hand_base_link, mass 0.06740077960995; collision mesh filename=meshes/right_hand/hand_base_link.STL; visual mesh filename=meshes/right_hand/hand_base_link.STL
- added link index_distal, mass 0.00376787129082313; collision mesh filename=meshes/right_hand/index_distal.STL; visual mesh filename=meshes/right_hand/index_distal.STL
- added link index_proximal, mass 0.00253178529301663; collision mesh filename=meshes/right_hand/index_proximal.STL; visual mesh filename=meshes/right_hand/index_proximal.STL
- added link index_tip
- added link middle_distal, mass 0.00376786259758948; collision mesh filename=meshes/right_hand/middle_distal.STL; visual mesh filename=meshes/right_hand/middle_distal.STL
- added link middle_proximal, mass 0.00253175497594429; collision mesh filename=meshes/right_hand/middle_proximal.STL; visual mesh filename=meshes/right_hand/middle_proximal.STL
- added link middle_tip
- added link pinky_distal, mass 0.00376782669873412; collision mesh filename=meshes/right_hand/pinky_distal.STL; visual mesh filename=meshes/right_hand/pinky_distal.STL
- added link pinky_proximal, mass 0.00253167400540778; collision mesh filename=meshes/right_hand/pinky_proximal.STL; visual mesh filename=meshes/right_hand/pinky_proximal.STL
- added link pinky_tip
- added link ring_distal, mass 0.0037678395356105; collision mesh filename=meshes/right_hand/ring_distal.STL; visual mesh filename=meshes/right_hand/ring_distal.STL
- added link ring_proximal, mass 0.00253170963529411; collision mesh filename=meshes/right_hand/ring_proximal.STL; visual mesh filename=meshes/right_hand/ring_proximal.STL
- added link ring_tip
- added link thumb_distal, mass 0.00763302603723749; collision mesh filename=meshes/right_hand/thumb_distal.STL; visual mesh filename=meshes/right_hand/thumb_distal.STL
- added link thumb_metacarpals, mass 0.0123381607727595; collision mesh filename=meshes/right_hand/thumb_metacarpals.STL; visual mesh filename=meshes/right_hand/thumb_metacarpals.STL
- added link thumb_metacarpals_base2, mass 0.00138591070212997; collision mesh filename=meshes/right_hand/thumb_metacarpals_base2.STL; visual mesh filename=meshes/right_hand/thumb_metacarpals_base2.STL
- added link thumb_tip
Joints:
- removed joint link_008_joint
- removed joint link_009_joint
- added joint index_dip: type revolute, parent index_proximal, child index_distal, origin xyz=-0.0052516 0 0.036625 rpy=0 0 0, axis 0 1 0, limit lower=0 upper=1.4 effort=100 velocity=1, mimic joint=index_mcp_pitch multiplier=0.89 offset=0
- added joint index_mcp_pitch: type revolute, parent hand_base_link, child index_proximal, origin xyz=0.0024758 0.02419 0.098779 rpy=-0.05236 0 0, axis 0 1 0, limit lower=0 upper=1.57 effort=100 velocity=1
- added joint index_tip_joint: type fixed, parent index_distal, child index_tip, origin xyz=0.016 0 0.035 rpy=0 0 0
- added joint link_007_to_hand: type fixed, parent link_007, child hand_base_link, origin xyz=0 0 -0.085 rpy=0 0 0
- added joint middle_dip: type revolute, parent middle_proximal, child middle_distal, origin xyz=-0.0052516 0 0.036625 rpy=0 0 0, axis 0 1 0, limit lower=0 upper=1.4 effort=100 velocity=1, mimic joint=middle_mcp_pitch multiplier=0.89 offset=0
- added joint middle_mcp_pitch: type revolute, parent hand_base_link, child middle_proximal, origin xyz=0.00052576 0.00634 0.1027 rpy=0 0 0, axis 0 1 0, limit lower=0 upper=1.57 effort=100 velocity=1
- added joint middle_tip_joint: type fixed, parent middle_distal, child middle_tip, origin xyz=0.016 0 0.035 rpy=0 0 0
- added joint pinky_dip: type revolute, parent pinky_proximal, child pinky_distal, origin xyz=-0.0052516 0 0.036625 rpy=0 0 0, axis 0 1 0, limit lower=0 upper=1.4 effort=100 velocity=1, mimic joint=pinky_mcp_pitch multiplier=0.89 offset=0
- added joint pinky_mcp_pitch: type revolute, parent hand_base_link, child pinky_proximal, origin xyz=0.0024758 -0.028372 0.092741 rpy=0.087266 0 0, axis 0 1 0, limit lower=0 upper=1.57 effort=100 velocity=1
- added joint pinky_tip_joint: type fixed, parent pinky_distal, child pinky_tip, origin xyz=0.016 0 0.035 rpy=0 0 0
- added joint ring_dip: type revolute, parent ring_proximal, child ring_distal, origin xyz=-0.0052516 0 0.036625 rpy=0 0 0, axis 0 1 0, limit lower=0 upper=1.4 effort=100 velocity=1, mimic joint=ring_mcp_pitch multiplier=0.89 offset=0
- added joint ring_mcp_pitch: type revolute, parent hand_base_link, child ring_proximal, origin xyz=0.0010258 -0.011135 0.098767 rpy=0.05236 0 0, axis 0 1 0, limit lower=0 upper=1.57 effort=100 velocity=1
- added joint ring_tip_joint: type fixed, parent ring_distal, child ring_tip, origin xyz=0.016 0 0.035 rpy=0 0 0
- added joint thumb_cmc_pitch: type revolute, parent thumb_metacarpals_base2, child thumb_metacarpals, origin xyz=0.0061649 0.010678 -0.004891 rpy=0 -1.1529 -2.0944, axis 0 1 0, limit lower=0 upper=0.52 effort=100 velocity=1
- added joint thumb_cmc_yaw: type revolute, parent hand_base_link, child thumb_metacarpals_base2, origin xyz=0.011508 0.022975 0.032794 rpy=0 0 0, axis 0 0 -1, limit lower=0 upper=1.54 effort=100 velocity=1
- added joint thumb_ip: type revolute, parent thumb_metacarpals, child thumb_distal, origin xyz=0.0037776 0 0.045368 rpy=0 0 0, axis 0 1 0, limit lower=0 upper=0.96 effort=100 velocity=1, mimic joint=thumb_cmc_pitch multiplier=1.83 offset=0
- added joint thumb_tip_joint: type fixed, parent thumb_distal, child thumb_tip, origin xyz=-0.002 0 0.044 rpy=0 0 0

Commit message: feat(urdf): mount the O6 hand on the JAKA flange adapter
Replace the placeholder link_007_to_hand pose with the real 45° adapter
supplied for the JAKA Mini flange. The STEP is tessellated to
urdf/meshes/adapter/jaka_o6_adapter.stl and inserted as
jaka_o6_adapter_link between link_007 and hand_base_link. The two
fixed-joint poses are derived from the adapter's real interfaces: 4×M6 on a
50 mm PCD to the flange and the O6's 20×20 mm M3 pattern to the hand. The
hand is clocked 270° about its bottom axis (90° + another 180°, equivalent
to -90°).

Drop the TG-9801 visuals that the JAKA app export left on link_007 (gripper
body, fingers and screws) so the model ends at the O6, and document the
mount and both 90°-symmetric clockings in the README, soma.yaml and the
URDF.

The hand chain itself is unchanged: its joint names match the primitive's
hand/info axes, and its layout agrees with the official linkerhand-urdf O6
right model to within ~2 mm.

Assisted-by: DeepSeek-Harness:deepseek-flash

File: urdf/robot.urdf (robot description, URDF)
Before this commit: robot generated_robot, 24 links, 23 joints
Links:
- added link jaka_o6_adapter_link, mass 0.224476; collision mesh filename=meshes/adapter/jaka_o6_adapter.stl; visual mesh filename=meshes/adapter/jaka_o6_adapter.stl
- link link_007: geometry collision mesh filename=meshes/part_006_solid_006.stl scale=0.001 0.001 0.001; collision mesh filename=meshes/part_007_solid_007.stl scale=0.001 0.001 0.001
Joints:
- removed joint link_007_to_hand
- added joint adapter_to_hand: type fixed, parent jaka_o6_adapter_link, child hand_base_link, origin xyz=0.000012 0.018631 -0.021738 rpy=0 0 4.712389
- added joint link_007_to_adapter: type fixed, parent link_007, child jaka_o6_adapter_link, origin xyz=0.0222186 -0.0341394 -0.0598598 rpy=2.3561945 0 -2.5649359
